Commit message: Nov 12 Modifications

File: src/CrazyS/rotors_description/urdf/crazyflie2.xacro (robot description, xacro)
@@ -18,25 +18,25 @@
 <robot name="crazyflie2" xmlns:xacro="http://ros.org/wiki/xacro">
   <!-- Properties (Taken from Novel Dynamic Inversion Architecture Design for Quadrocopter Control by Jian Wang et al.) -->
-  <xacro:property name="namespace" value="$(arg namespace)" />
-  <xacro:property name="rotor_velocity_slowdown_sim" value="50" />
-  <xacro:property name="use_mesh_file" value="true" />
-  <xacro:property name="mesh_file" value="package://rotors_description/meshes/crazyflie2.dae" />
-  <xacro:property name="mass" value="0.025" /> <!-- [kg] -->
-  <xacro:property name="body_width" value="0.045" /> <!-- [m] -->
-  <xacro:property name="body_height" value="0.03" /> <!-- [m] -->
-  <xacro:property name="mass_rotor" value="0.0005" /> <!-- [kg] -->
-  <xacro:property name="arm_length" value="0.046" /> <!-- [m] -->
-  <xacro:property name="rotor_offset_top" value="0.024" /> <!-- [m] -->
-  <xacro:property name="radius_rotor" value="0.0225" /> <!-- [m] -->
-  <xacro:property name="sin45" value="0.707106781186" />
-  <xacro:property name="cos45" value="0.707106781186" />
-  <!-- Forster's -->
-  <xacro:property name="motor_constant" value="1.28192e-08" /> <!-- [kg m/s^2] -->
-  <xacro:property name="moment_constant" value="5.964552e-03" /> <!-- [m] -->
-  <xacro:property name="time_constant_up" value="0.0125" /> <!-- [s] -->
-  <xacro:property name="time_constant_down" value="0.025" /> <!-- [s] -->
-  <xacro:property name="max_rot_velocity" value="2618" /> <!-- [rad/s] -->
-  <xacro:property name="rotor_drag_coefficient" value="8.06428e-05" />
-  <xacro:property name="rolling_moment_coefficient" value="0.000001" />
+    <xacro:property name="namespace" value="$(arg namespace)" />
+    <xacro:property name="rotor_velocity_slowdown_sim" value="50" />
+    <xacro:property name="use_mesh_file" value="true" />
+    <xacro:property name="mesh_file" value="package://rotors_description/meshes/crazyflie2.dae" />
+    <xacro:property name="mass" value="0.025" /> <!-- [kg] -->
+    <xacro:property name="body_width" value="0.045" /> <!-- [m] -->
+    <xacro:property name="body_height" value="0.03" /> <!-- [m] -->
+    <xacro:property name="mass_rotor" value="0.0005" /> <!-- [kg] -->
+    <xacro:property name="arm_length" value="0.046" /> <!-- [m] -->
+    <xacro:property name="rotor_offset_top" value="0.024" /> <!-- [m] -->
+    <xacro:property name="radius_rotor" value="0.0225" /> <!-- [m] -->
+    <xacro:property name="sin45" value="0.707106781186" />
+    <xacro:property name="cos45" value="0.707106781186" />
+    <!-- Forster's -->
+    <xacro:property name="motor_constant" value="1.28192e-08" /> <!-- [kg m/s^2] -->
+    <xacro:property name="moment_constant" value="5.964552e-03" /> <!-- [m] -->
+    <xacro:property name="time_constant_up" value="0.0125" /> <!-- [s] -->
+    <xacro:property name="time_constant_down" value="0.025" /> <!-- [s] -->
+    <xacro:property name="max_rot_velocity" value="2618" /> <!-- [rad/s] -->
+    <xacro:property name="rotor_drag_coefficient" value="8.06428e-05" />
+    <xacro:property name="rolling_moment_coefficient" value="0.000001" />
   <!-- Property Blocks -->
   <xacro:property name="body_inertia">
